File: LNWBA.kicad_sch (KiCad schematic)
At the start: 2 parts, among them Q1 JFE2140D, Q2 2N3904

Commit message: Ki..
Parts:
- added R1, R2: 2k, symbol Device:R_US
Connections:
- net at Q1.2: now also R1.2
- net at Q1.6: now also R2.2
- new net +15V: R1.1, R2.1
