File: LNWBA.kicad_sch (KiCad schematic)
At the start: 4 parts, among them Q1 JFE2140D, Q2 2N3904

Commit message: BJT?
Parts:
- added C1: 0pF, Capacitor_SMD:C_0603_1608Metric_Pad1.08x0.95mm_HandSolder, symbol Device:C
- added C2: 2pF, Capacitor_SMD:C_0603_1608Metric_Pad1.08x0.95mm_HandSolder, symbol Device:C
- added R12: 2k, Resistor_SMD:R_0603_1608Metric_Pad0.98x0.95mm_HandSolder, symbol Device:R_US
- added R13, R4: 10k, Resistor_SMD:R_0603_1608Metric_Pad0.98x0.95mm_HandSolder, symbol Device:R_US
- added R14: 100, Resistor_SMD:R_0603_1608Metric_Pad0.98x0.95mm_HandSolder, symbol Device:R_US
- added R3, R7: 100k, Resistor_SMD:R_0603_1608Metric_Pad0.98x0.95mm_HandSolder, symbol Device:R_US
- added R5: 1k, Resistor_SMD:R_0603_1608Metric_Pad0.98x0.95mm_HandSolder, symbol Device:R_US
- added R6: 1M, Resistor_SMD:R_0603_1608Metric_Pad0.98x0.95mm_HandSolder, symbol Device:R_US
- added U1, U3: LM7171xIM, Package_SO:SOIC-8_3.9x4.9mm_P1.27mm, symbol Amplifier_Operational:LM7171xIM
- added U2: NC7SB3157P6X, Package_TO_SOT_SMD:SOT-363_SC-70-6_Handsoldering, symbol Analog_Switch:NC7SB3157P6X
- R1, R2: footprint (none) -> Resistor_SMD:R_0603_1608Metric_Pad0.98x0.95mm_HandSolder
Connections:
- net +15V: now also U1.7 (V+), U3.7 (V+)
- net at Q1.2, R1.2: now also U1.2 (-)
- net at Q2.1 (E): now also R12.1
- net at Q1.6, R2.2: now also U1.3 (+)
- net at Q1.8: now also U2.4
- new net: C2.1, R14.2, R4.1, R5.1, R7.1, U2.1
- new net: C1.1, C2.2, R13.1, R3.1, R4.2, R5.2, R6.1, R7.2, U2.3
- new net: C1.2, R13.2, R3.2, R6.2, U1.6, U3.3 (+)
- new net -15V: R12.2, U1.4 (V-), U3.4 (V-)
- new net GND: R14.1
